File: makeFlash.kicad_pcb (KiCad board)
At the start: 2 copper layers, 48.3 x 78.7 mm, 15 parts, among them Q1 2N3904, Q2 2N3904

Commit message: FAB Ready Version?
Parts:
- added KiCadLogo: KiCad-Logo2_6mm_SilkScreen, Symbols:KiCad-Logo2_6mm_SilkScreen, F.Cu at (218.4, 101.6)
- added REF***: OSHW-Logo2_9.8x8mm_SilkScreen, Symbols:OSHW-Logo2_9.8x8mm_SilkScreen, F.Cu at (218.4, 115.6)
Other:
- net class Default: clearance 0.2 -> 0.4
- rule trace_clearance: 0.2 -> 0.4
- board text added: "http://github.com/splatski/makeFlash"
